File: Layer2/Layer2/Layer2.kicad_pcb (KiCad board)
At the start: 2 copper layers, 99.9 x 99.9 mm, 34 parts, among them J1 Conn_02x20_Odd_Even, J2 Conn_02x20_Odd_Even, U1 74LS08, U10 74HC245, U11 74HC245, U12 74LS181, U13 28C256, U14 74LS173, U15 628128_DIP32_SSOP32, U16 74LS173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

Commit message: Layer 3 complete
Parts:
- moved C8 172.4 mm to (20.9, 109.0), turned to 90 degrees
- moved C9 133.8 mm to (66.1, 102.7), turned to 180 degrees
- moved C6 83.5 mm to (112.1, 107.5)
- moved U18 0.39 mm to (40.3, 110.6)
Connections:
- J1 pad 24: Bank_Reg_In -> CU_CtrlLn16
- J2 pad 29: CU_CtrlLn23 -> Bank_Reg_In
- U13 pad 22: CU_MuEx_CtrlLn5 -> CU_MuEx_CtrlLn10
- U15 pad 24: CU_MuEx_CtrlLn5 -> CU_MuEx_CtrlLn10
- U17 pad 3: Net-(U17-Pad3) -> GND
- U17 pad 4: Net-(U17-Pad3) -> GND
- U17 pad 8: Net-(U17-Pad3) -> GND
Routing:
- net Bus_6: track 267.0 -> 415.2 mm, vias 0 -> 1
- net CU_MuEx_CtrlLn10: track 0.00 -> 141.0 mm, vias 0 -> 1
- net CLK_OUT: track 178.5 -> 310.6 mm, vias 1 -> 2
- net Bus_5: track 264.9 -> 384.3 mm, vias 0 -> 2
- net Bus_7: track 261.2 -> 373.5 mm, vias 1 -> 5
- net Bus_4: track 234.3 -> 343.1 mm, vias 0 -> 1
- net GND: track 111.9 -> 205.9 mm, vias 5 -> 11
- net EEPROM_CS: track 0.71 -> 92.7 mm, vias 0 -> 1
- net Bus_0: track 251.1 -> 343.0 mm, vias 0 -> 2
- net Ram_CS: track 2.59 -> 89.0 mm, vias 0 -> 2
- net Bus_2: track 256.6 -> 331.5 mm, vias 0 -> 1
- net Net-(U16-Pad6): track 0.00 -> 73.2 mm
- net Bus_1: track 259.7 -> 328.0 mm, vias 0 -> 1
- net Net-(U16-Pad5): track 0.00 -> 65.8 mm
- net M_RST: track 296.0 -> 361.7 mm, vias 1 -> 2
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- added copper zone on B.Cu, net +5V
