File: Layer3/Layer3/Layer3-backup.sch (KiCad schematic (older format))
At the start: 48 parts, among them IC1 74HCT4060D-Q100,11, J1 Conn_02x20_Odd_Even, J2 Conn_02x20_Odd_Even, J3 Conn_02x12_Odd_Even, J4 Barrel_Jack_MountingPin, Q1 2N2222, SW1 SW_Push, SW2 SW_Push, SW3 SW_DIP_x01, U1 28C256, U10 7400, U11 NE555, U2 74LS193, U3 74461, U4 28C256, U5 74154, U6 74461, U7 28C256, U8 74HCT273, U9 28C256, X1 SG-8002DC

Commit message: Layer 3 complete
Parts:
- added J?: DB15_Female_HighDensity_MountingHoles, symbol Connector:DB15_Female_HighDensity_MountingHoles
- added U?: IDT7132, symbol Memory_RAM:IDT7132
- added U?: 74LS595, symbol 74xx:74LS595
- added U? (x2): IDT7130, symbol Memory_RAM:IDT7132
- added U?: 74LS157, symbol 74xx:74LS157
- added U? (x3): 4040, symbol 4xxx:4040
- added U?: 28C256, symbol Memory_EEPROM:28C256
- added X?: SG-8002DC, Oscillator:Oscillator_SeikoEpson_SG-8002DC, symbol Oscillator:SG-8002DC
- renumbered C10 to C?, C2 to C?, C3 to C?, C4 to C?, C5 to C?, C6 to C?, C7 to C?, C8 to C?, C9 to C?, C12 to C?, C13 to C?, C11 to C?, C1 to C?, H4 to H?, H3 to H?, H2 to H?, H1 to H?, IC1 to IC?, J3 to J?, J4 to J?, J1 to J?, J2 to J?, Q1 to Q?, R4 to R?, R6 to R?, R3 to R?, R5 to R?, R7 to R?, R1 to R?, R2 to R?, R9 to R?, R8 to R?, RV1 to RV?, SW2 to SW?, SW3 to SW?, SW1 to SW?, U1 to U?, U4 to U?, U7 to U?, U9 to U?, U2 to U?, U5 to U?, U11 to U?, U10 to U?, U8 to U?, U3 to U?, U6 to U?, X1 to X?
Connections:
- net BTN_OUT is gone; now on net +5V: C?.1, R?.1, U?.13
- net GND is gone; now on net +5V: C?.2, C?.2, C?.2, C?.2, C?.2, C?.2, C?.2, C?.2, C?.2, C?.2, C?.2, C?.2, C?.2, IC?.12, IC?.8, J?.2, J?.39 (Pin_39), J?.40 (Pin_40), Q?.1 (E), SW?.1, SW?.1, SW?.1, U?.1 (GND), U?.10 (GND), U?.12 (GND), U?.12 (GND), U?.12 (GND), U?.14 (GND), U?.14 (GND), U?.14 (GND), U?.14 (GND), U?.18 (~E0), U?.19 (~E1), U?.20 (~CS), U?.20 (~CS), U?.20 (~CS), U?.20 (~CS), U?.22 (~OE), U?.22 (~OE), U?.22 (~OE), U?.22 (~OE), U?.23 (CI), U?.7 (GND), U?.8 (GND), X?.4 (GND)
- net Switch_OUT is gone; now on net +5V: C?.1, R?.1, U?.1, U?.12, U?.2
- net +5V: now also IC?.4, J?.18 (Pin_18), R?.2, R?.2, SW?.2, U?.1 (A14), U?.1 (A14), U?.1 (A14), U?.1 (A14), U?.1 (/CEL), U?.1 (/CEL), U?.1 (/CEL), U?.12 (RCLK), U?.14 (GND), U?.16 (VCC), U?.16 (VDD), U?.16 (VDD), U?.2 (R/WL), U?.2 (R/WL), U?.2 (R/WL), U?.20 (~CS), U?.22 (~OE), U?.24 (GND), U?.24 (GND), U?.24 (GND), U?.27 (~WE), U?.28 (VCC), U?.4 (Za), U?.48 (VCC), U?.48 (VCC), U?.48 (VCC), U?.5 (/OEL), U?.5 (/OEL), U?.5 (/OEL), U?.6 (A0L), U?.6 (A0L), U?.8 (GND), U?.8 (GND), U?.8 (VSS), U?.8 (VSS), U?.8 (VSS), U?.9 (Q0), X?.1 (OE), X?.4 (GND), X?.8 (Vcc)
- net Bus_0: now also U?.12 (Zd)
- net HC_RST: now reaches IC?.14, J?.14 (Pin_14)
- net HC_RST: now also U?.11 (D0), U?.11 (Reset)
- removed net KF: J?.23 (Pin_23), U?.1 (A14), U?.1 (A14), U?.1 (A14), U?.1 (A14)
- new net ChrC_CLK: U?.10 (CLK), U?.16 (D4)
- new net ChrC_RST: U?.11 (Reset), U?.15 (D3)
- new net Chr_Col_0: U?.7 (Q1)
- new net Chr_Col_1: U?.6 (Q2)
- new net Chr_Col_2: U?.5 (Q3)
- new net Chr_Row_0: U?.3 (A7), U?.6 (A0L), U?.7 (Q1)
- new net Chr_Row_1: U?.25 (A8), U?.6 (Q2), U?.7 (A1L)
- new net Chr_Row_2: U?.24 (A9), U?.5 (Q3), U?.8 (A2L)
- new net Cur_Chr_Code_0: U?.16 (I/O0L), U?.9 (A3L)
- new net Cur_Chr_Code_1: U?.10 (A4L), U?.17 (I/O1L)
- new net Cur_Chr_Code_2: U?.11 (A5L), U?.18 (I/O2L)
- new net Cur_Chr_Code_3: U?.12 (A6L), U?.19 (I/O3L)
- new net Cur_Chr_Code_4: U?.13 (A7L), U?.20 (I/O4L)
- new net Cur_Chr_Code_5: U?.14 (A8L), U?.21 (I/O5L)
- new net Cur_Chr_Code_6: U?.15 (A9L), U?.22 (I/O6L)
- new net Cur_Chr_Code_7: U?.23 (I/O7L), U?.4 (A10L)
- new net Cur_Color_1: U?.7 (Zb)
- new net Cur_Color_2: U?.9 (Zc)
- new net Cur_Color_Opt1_0: U?.16 (I/O0L), U?.2 (I0a)
- new net Cur_Color_Opt1_1: U?.17 (I/O1L), U?.5 (I0b)
- new net Cur_Color_Opt1_2: U?.11 (I0c), U?.18 (I/O2L)
- new net Cur_Color_Opt1_3: U?.14 (I0d), U?.19 (I/O3L)
- new net Cur_Color_Opt2_0: U?.20 (I/O4L), U?.3 (I1a)
- new net Cur_Color_Opt2_1: U?.21 (I/O5L), U?.6 (I1b)
- new net Cur_Color_Opt2_2: U?.10 (I1c), U?.22 (I/O6L)
- new net Cur_Color_Opt2_3: U?.13 (I1d), U?.23 (I/O7L)
- new net Cur_Color_Sel: U?.1 (S), U?.9 (QH')
- new net Cur_Row_Color_Sel_0: U?.16 (I/O0L), U?.7 (QH)
- new net Cur_Row_Color_Sel_1: U?.17 (I/O1L), U?.6 (QG)
- new net Cur_Row_Color_Sel_2: U?.18 (I/O2L), U?.5 (QF)
- new net Cur_Row_Color_Sel_3: U?.19 (I/O3L), U?.4 (QE)
- new net Cur_Row_Color_Sel_4: U?.20 (I/O4L), U?.3 (QD)
- new net Cur_Row_Color_Sel_5: U?.2 (QC), U?.21 (I/O5L)
- new net Cur_Row_Color_Sel_6: U?.1 (QB), U?.22 (I/O6L)
- new net Cur_Row_Color_Sel_7: U?.15 (QA), U?.23 (I/O7L)
- new net HC_0: U?.10 (A0), U?.3 (Q4)
- new net HC_1: U?.2 (Q5), U?.9 (A1)
- new net HC_2: U?.4 (Q6), U?.8 (A2)
- new net HC_3: U?.13 (Q7), U?.7 (A3)
- new net HC_4: U?.12 (Q8), U?.6 (A4)
- new net HC_5: U?.14 (Q9), U?.5 (A5)
- new net PXL_CLK: U?.10 (CLK), X?.5 (OUT)
- new net Porch_Active: U?.15 (E), U?.17 (D5)
- new net VC_0: U?.4 (A6), U?.9 (Q0)
- new net VC_1: U?.21 (A10), U?.3 (Q4)
- new net VC_2: U?.2 (Q5), U?.23 (A11)
- new net VC_3: U?.2 (A12), U?.4 (Q6)
- new net VC_4: U?.13 (Q7), U?.26 (A13)
- new net VC_5: U?.1 (A14), U?.12 (Q8)
- new net VC_CLK: U?.10 (CLK), U?.13 (D2)
- new net VC_RST: U?.11 (Reset), U?.12 (D1)
- new net V_Mem_Add_1: U?.7 (A1L), U?.7 (A1L), U?.7 (Q1)
- new net V_Mem_Add_2: U?.6 (Q2), U?.8 (A2L), U?.8 (A2L)
- new net V_Mem_Add_3: U?.5 (Q3), U?.9 (A3L), U?.9 (A3L)
- new net V_Mem_Add_4: U?.10 (A4L), U?.10 (A4L), U?.3 (Q4)
- new net V_Mem_Add_5: U?.11 (A5L), U?.11 (A5L), U?.2 (Q5)
- new net V_Mem_Add_6: U?.12 (A6L), U?.12 (A6L), U?.4 (Q6)
- new net V_Mem_Add_7: U?.13 (A7L), U?.13 (A7L), U?.13 (Q7)
- new net V_Mem_Add_8: U?.12 (Q8), U?.14 (A8L), U?.14 (A8L)
- new net V_Mem_Add_9: U?.14 (Q9), U?.15 (A9L), U?.15 (A9L)
