File: Layer3/Layer3/Layer3.kicad_pcb (KiCad board)
At the start: 2 copper layers, 99.9 x 99.9 mm, 37 parts, among them J1 Conn_02x20_Odd_Even, J2 Conn_02x20_Odd_Even, J3 DB15_Female_HighDensity_Mount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, U1 74LS165, U10 74LS00, U11 28C256, U12 IDT7130, U2 74LS157, U3 74461, U4 4040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

Commit message: Backup
Parts:
- moved C8 17.9 mm to (53.0, 114.8), turned to 270 degrees
Routing:
- net VRAM_Add_10: track 187.1 -> 188.2 mm
