File: Layer3/Layer3/Layer3.sch (KiCad schematic (older format))
At the start: 37 parts, among them J1 Conn_02x20_Odd_Even, J2 Conn_02x20_Odd_Even, J3 DB15_Female_HighDensity_Mount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, U1 74LS165, U10 74LS00, U11 28C256, U12 IDT7130, U2 74LS157, U3 74461, U4 4040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

Commit message: Backup
Parts:
- J3: footprint (none) -> Connector_Dsub:DSUB-15-HD_Female_Horizontal_P2.29x1.98mm_EdgePinOffset3.03mm_Housed_MountingHolesOffset4.94mm
Changed lines of the file:
@@
 F 0 "J3" H 1100 7717 50  0000 C CNN
 F 1 "DB15_Female_HighDensity_MountingHoles" H 1100 7626 50  0000 C CNN
-F 2 "" H 150 7250 50  0001 C CNN
+F 2 "Connector_Dsub:DSUB-15-HD_Female_Horizontal_P2.29x1.98mm_EdgePinOffset3.03mm_Housed_MountingHolesOffset4.94mm" H 150 7250 50  0001 C CNN
 F 3 " ~" H 150 7250 50  0001 C CNN
 	1    1100 6850
