File: Layer1/Layer1.kicad_pcb (KiCad board)
At the start: 2 copper layers, 99.9 x 99.9 mm, 45 parts, among them IC1 74HCT4060D-Q100,11, J1 Conn_02x20_Odd_Even, J2 Conn_02x20_Odd_Even, J3 Conn_02x12_Odd_Even, J4 Barrel_Jack_MountingPin, SW1 SW_Push, SW2 SW_Push, SW3 SW_DIP_x01, U1 28C256, U10 7400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

Commit message: Finished Layer1
Parts:
- moved C5 129.9 mm to (27.5, 39.3), turned to 90 degrees
- moved C8 113.8 mm to (72.5, 29.8)
- moved C13 110.8 mm to (26.3, 99.7)
- moved C7 105.9 mm to (103.5, 23.7)
- moved C12 86.3 mm to (50.7, 106.5)
- moved C6 73.5 mm to (75.5, 65.9), turned to 180 degrees
- moved C4 60.3 mm to (108.4, 79.8), turned to 90 degrees
- moved C9 35.2 mm to (112.3, 96.9)
- moved U10 0.36 mm to (101.2, 107.4)
Connections:
- J1 pad 10: Net-(J1-Pad10) -> CU_CtrlLn7
- J1 pad 12: Net-(J1-Pad12) -> CU_CtrlLn6
- J1 pad 14: Net-(J1-Pad14) -> CU_CtrlLn5
- J1 pad 16: Net-(J1-Pad16) -> CU_CtrlLn12
- J1 pad 18: Net-(J1-Pad18) -> CU_CtrlLn13
- J1 pad 2: Net-(J1-Pad2) -> CU_CtrlLn11
- J1 pad 20: Net-(J1-Pad20) -> CU_CtrlLn14
- J1 pad 22: Net-(J1-Pad22) -> CU_CtrlLn15
- J1 pad 24: Net-(J1-Pad24) -> CU_CtrlLn16
- J1 pad 26: Net-(J1-Pad26) -> CU_CtrlLn17
- J1 pad 28: Net-(J1-Pad28) -> CU_CtrlLn18
- J1 pad 30: Net-(J1-Pad30) -> CU_CtrlLn19
- J1 pad 4: Net-(J1-Pad4) -> CU_CtrlLn10
- J1 pad 6: Net-(J1-Pad6) -> CU_CtrlLn9
- J1 pad 8: Net-(J1-Pad8) -> CU_CtrlLn8
- J2 pad 29: Net-(J2-Pad29) -> CU_CtrlLn23
- J2 pad 31: Net-(J2-Pad31) -> CU_CtrlLn24
- J2 pad 35: Net-(J2-Pad35) -> CU_CtrlLn20
- J2 pad 37: Net-(J2-Pad37) -> CU_CtrlLn21
- J2 pad 39: Net-(J2-Pad39) -> CU_CtrlLn22
Routing:
- net +5V: track 0.00 -> 173.1 mm, vias 0 -> 1
- net GND: track 0.00 -> 157.9 mm
- net Bus_4: track 41.7 -> 134.6 mm, vias 0 -> 1
- net CU_MuEx_CtrlLn14: track 0.00 -> 89.1 mm
- net Bus_5: track 41.7 -> 123.1 mm, vias 0 -> 1
- net Bus_7: track 36.8 -> 104.7 mm, vias 0 -> 2
- net Bus_6: track 36.8 -> 103.1 mm, vias 0 -> 2
- net Bus_0: track 61.6 -> 123.3 mm, vias 0 -> 1
- net Bus_1: track 56.0 -> 112.9 mm, vias 0 -> 1
- net Bus_2: track 51.5 -> 104.6 mm, vias 0 -> 1
- net Bus_3: track 45.4 -> 97.7 mm, vias 0 -> 1
- net CU_CtrlLn7: track 0.00 -> 49.7 mm
- net Net-(U3-Pad14): track 0.00 -> 48.3 mm
- net CU_CtrlLn23: track 0.00 -> 47.6 mm
- net CU_CtrlLn6: track 0.00 -> 46.2 mm
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
Commit message: Layer2 Progress
Parts:
- added Q1: 2N2222, Package_TO_SOT_THT:TO-92, F.Cu at (78.7, 72.4)
- added R8: 10k, Resistor_THT:R_Axial_DIN0309_L9.0mm_D3.2mm_P12.70mm_Horizontal, F.Cu at (20.8, 96.5)
- added R9: 1k, Resistor_THT:R_Axial_DIN0309_L9.0mm_D3.2mm_P12.70mm_Horizontal, F.Cu at (49.3, 117.9)
- moved C12 3.34 mm to (53.8, 105.4)
- moved C13 2.13 mm to (26.3, 97.5)
Connections:
- J2 pad 25: Net-(J2-Pad25) -> EF
- J2 pad 27: Net-(J2-Pad27) -> CF
- U1 pad 2: CE -> EF
- U2 pad 5: CLK_OUT -> Net-(Q1-Pad3)
- U4 pad 2: CE -> EF
- U7 pad 2: CE -> EF
- U9 pad 2: CE -> EF
Routing:
- net EF: track 0.00 -> 161.8 mm
- net CE: track 160.4 -> 0.00 mm
- net Net-(Q1-Pad2): track 0.00 -> 87.6 mm
- net Net-(Q1-Pad3): track 0.00 -> 76.2 mm
- net CLK_OUT: track 248.2 -> 208.8 mm, vias 1 -> 0
- net I_6: track 188.8 -> 179.1 mm
- net I_7: track 167.6 -> 171.8 mm
- net +5V: track 173.1 -> 174.8 mm
- net I_3: track 121.8 -> 123.5 mm
- net M_RST: track 215.0 -> 216.5 mm
- net CF: track 191.6 -> 192.6 mm
- net GND: track 157.9 -> 157.0 mm
- net I_0: track 181.2 -> 181.7 mm

Commit message: Layer 3 complete
Connections:
- J2 pad 23: Net-(J2-Pad23) -> KF
- U1 pad 1: GND -> KF
Routing:
- net KF: track 0.00 -> 57.0 mm
- net I_7: track 171.8 -> 178.2 mm
- net GND: track 157.0 -> 151.6 mm
- net I_5: track 154.2 -> 159.4 mm
- net CF: track 192.6 -> 197.6 mm
- net EF: track 161.8 -> 165.6 mm
- net I_6: track 179.1 -> 182.5 mm
- net +5V: track 174.8 -> 177.2 mm
- net I_1: track 165.5 -> 164.3 mm
- net I_2: track 160.0 -> 158.8 mm
- net I_4: track 135.8 -> 136.9 mm
- net I_0: track 181.7 -> 181.2 mm

Commit message: Backup
Parts:
- removed Q1: 2N2222, Package_TO_SOT_THT:TO-92
- removed R8: 10k, Resistor_THT:R_Axial_DIN0309_L9.0mm_D3.2mm_P12.70mm_Horizontal
- removed R9: 1k, Resistor_THT:R_Axial_DIN0309_L9.0mm_D3.2mm_P12.70mm_Horizontal
- added U12: 74LS04, Package_DIP:DIP-14_W7.62mm_LongPads, F.Cu at (184.8, 73.6)
- added U12: 74HC804, Package_DIP:DIP-20_W7.62mm_LongPads, F.Cu at (93.6, 107.5)
- added U13: 74LS02, Package_DIP:DIP-14_W7.62mm_LongPads, F.Cu at (196.4, 51.7)
- added U14: 74LS00, Package_DIP:DIP-14_W7.62mm_LongPads, F.Cu at (208.0, 51.7)
- added U15: 74LS02, Package_DIP:DIP-14_W7.62mm_LongPads, F.Cu at (219.6, 51.7)
- added U16: 74LS04, Package_DIP:DIP-14_W7.62mm_LongPads, F.Cu at (196.4, 71.1)
- added U17: 74LS02, Package_DIP:DIP-14_W7.62mm_LongPads, F.Cu at (208.0, 71.1)
- added U18: 74LS08, Package_DIP:DIP-14_W7.62mm_LongPads, F.Cu at (219.6, 71.1)
- added U19: 74LS00, Package_DIP:DIP-14_W7.62mm_LongPads, F.Cu at (231.2, 51.7)
- added U20: 74LS04, Package_DIP:DIP-14_W7.62mm_LongPads, F.Cu at (231.2, 71.1)
- added U21: SST39SF010, Package_DIP:DIP-32_W15.24mm_LongPads, F.Cu at (154.0, 51.7)
- added U22: 74HC238, Package_DIP:DIP-16_W7.62mm_LongPads, F.Cu at (173.2, 51.7)
- added U23: 74LS138, Package_DIP:DIP-16_W7.62mm_LongPads, F.Cu at (184.8, 51.7)
- U10: value 7400 -> 74LS08; footprint Package_DIP:DIP-14_W7.62mm -> Package_DIP:DIP-14_W7.62mm_LongPads
- moved U10 79.5 mm to (173.2, 73.6), turned to 0 degrees
- moved R4 16.0 mm to (70.2, 98.8)
- moved C9 5.83 mm to (106.5, 96.1)
- moved RV1 5.23 mm to (73.5, 116.3)
- moved SW3 5.23 mm to (81.2, 117.4)
- moved U11 5.23 mm to (58.8, 117.2)
- moved C12 5.23 mm to (48.6, 105.5)
- moved C2 5.23 mm to (61.2, 106.2)
- moved C3 5.23 mm to (50.8, 115.6)
- moved R3 5.23 mm to (54.9, 117.7)
- moved R6 5.15 mm to (86.0, 111.3), turned to 90 degrees
- moved R7 0.76 mm to (70.2, 102.6)
- moved R5 0.49 mm to (70.2, 106.4)
- moved C4 0.31 mm to (108.7, 79.9)
Connections:
- net CU_CtrlLn7 renamed ALU_M
- net CU_MuExCtrlM_0 renamed CU_MuExCtrlOut_0
- net CU_MuExCtrlM_1 renamed CU_MuExCtrlOut_1
- net CU_MuExCtrlM_2 renamed CU_MuExCtrlOut_2
- net CU_MuExCtrlM_3 renamed CU_MuExCtrlOut_3
- net CU_MuEx_CtrlLn0 renamed Net-(U5-Pad1)
- net CU_MuEx_CtrlLn1 renamed SP_OE
- net CU_MuEx_CtrlLn15 renamed Net-(U5-Pad17)
- net I_Reg_LD renamed Net-(U8-Pad11)
- J1 pad 3: Net-(J1-Pad3) -> CU_C0
- J1 pad 31: Net-(J1-Pad31) -> I_0
- J1 pad 32: Net-(J1-Pad32) -> I_4
- J1 pad 33: Net-(J1-Pad33) -> I_1
- J1 pad 34: Net-(J1-Pad34) -> I_5
- J1 pad 35: Net-(J1-Pad35) -> I_2
- J1 pad 36: Net-(J1-Pad36) -> I_6
- J1 pad 37: Net-(J1-Pad37) -> I_3
- J1 pad 38: Net-(J1-Pad38) -> I_7
- J1 pad 5: Net-(J1-Pad5) -> CU_C1
- J1 pad 7: Net-(J1-Pad7) -> CU_C2
- J1 pad 9: Net-(J1-Pad9) -> CU_C3
- U1 pad 1: KF -> M_RST
- U1 pad 3: I_7 -> KF
- U1 pad 4: I_6 -> Net-(U1-Pad4)
- U10 pad 1: Switch_OUT -> CU_CtrlLn3
- U10 pad 10: Net-(U10-Pad10) -> Counter_Countrol_Inverted
- U10 pad 11: Net-(U10-Pad10) -> Net-(U10-Pad11)
- U10 pad 12: Switch_OUT -> CU_CtrlLn0
- U10 pad 13: BTN_OUT -> Counter_Countrol_Inverted
- U10 pad 2: Switch_OUT -> Counter_Countrol_Inverted
- U10 pad 4: 555_OUT -> CU_CtrlLn2
- U10 pad 5: Net-(U10-Pad3) -> Counter_Countrol_Inverted
- U10 pad 8: Debug_CLK_OUT -> Net-(U10-Pad8)
- U10 pad 9: Net-(U10-Pad6) -> CU_CtrlLn1
- U2 pad 14: M_RST -> CU_CtrlLn27
- U4 pad 1: GND -> M_RST
- U5 pad 10: CU_MuEx_CtrlLn9 -> VRam_OE
- U5 pad 11: CU_MuEx_CtrlLn10 -> PS2_Out
- U5 pad 13: CU_MuEx_CtrlLn11 -> Counter_Control
- U5 pad 14: CU_MuEx_CtrlLn12 -> Net-(U5-Pad14)
- U5 pad 15: CU_MuEx_CtrlLn13 -> Net-(U5-Pad15)
- U5 pad 16: CU_MuEx_CtrlLn14 -> Net-(U5-Pad16)
- U5 pad 18: GND -> ALU_Out
- U5 pad 3: CU_MuEx_CtrlLn2 -> PC_L_OE
- U5 pad 4: CU_MuEx_CtrlLn3 -> PC_H_OE
- U5 pad 5: CU_MuEx_CtrlLn4 -> A_Out
- U5 pad 6: CU_MuEx_CtrlLn5 -> B_Out
- U5 pad 7: CU_MuEx_CtrlLn6 -> Net-(U18-Pad4)
- U5 pad 8: CU_MuEx_CtrlLn7 -> D_Out
- U5 pad 9: CU_MuEx_CtrlLn8 -> Ram_Out
- U7 pad 1: GND -> M_RST
- U9 pad 1: GND -> M_RST
Routing:
- net Net-(U1-Pad4): track 0.00 -> 157.9 mm
- net Net-(U12-Pad3): track 0.00 -> 143.5 mm
- net M_RST: track 216.5 -> 337.8 mm, vias 1 -> 0
- net I_6: track 182.5 -> 272.3 mm
- net Net-(Q1-Pad2): track 87.6 -> 0.00 mm
- net Net-(U16-Pad10): track 76.2 -> 0.00 mm
- net CU_C2: track 167.4 -> 225.9 mm
- net I_3: track 123.5 -> 172.4 mm
- net GND: track 151.6 -> 103.6 mm, vias 0 -> 2
- net I_2: track 158.8 -> 205.0 mm
- net CU_C3: track 170.3 -> 211.5 mm
- net CU_C1: track 144.1 -> 182.1 mm
- net CLK_OUT: track 208.8 -> 245.9 mm
- net CU_CtrlLn27: track 36.7 -> 70.6 mm, vias 0 -> 1
- net I_5: track 159.4 -> 193.2 mm
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